File: hw/sch_pcb/VLFANT01A.kicad_pcb (KiCad board)
At the start: 2 copper layers, 50.3 x 40.1 mm, 19 parts, among them J1 CONN_3, J2 CONN_3, J3 CONN_3, J4 CONN_3, J5 CONN_3, J6 CONN_3, J7 SMA, J8 CONN_3, J9 JUMP_3X2, M1 HOLE, M10 HOLE, M2 HOLE, M3 HOLE, M4 HOLE, M5 HOLE, M6 HOLE, M7 HOLE, M8 HOLE, M9 HOLE

Commit message: update to new kicad format
Other:
- net class Default removed
