File: hw/sch_pcb/VLFANT01B.kicad_pcb (KiCad board)
At the start: 2 copper layers, 50.3 x 40.1 mm, 9 parts, among them J1 RJ45_RJHSE-5384, J2 RJ45_RJHSE-5384, J3 RJ45_RJHSE-5384, J7 SMA, J9 JUMP_3X2, M1 HOLE, M2 HOLE, M3 HOLE, M4 HOLE

Commit message: verze s narazecimi konektory
Parts:
- added J4: JUMP_2x1, Mlab_Pin_Headers:Straight_1x01, F.Cu at (154.5, 88.2)
- added J5: IDC381-8-110, Mlab_CON:IDC381-8-110, F.Cu at (154.6, 106.0)
- added J6: JUMP_2x1, Mlab_Pin_Headers:Straight_1x01, F.Cu at (161.6, 122.4)
- J1, J3: value RJ45_RJHSE-5384 -> IDC381-8-110; footprint Mlab_CON:RJHSE-5384(RJ45) -> Mlab_CON:IDC381-8-110
- J2: value RJ45_RJHSE-5384 -> JUMP_2x1; footprint Mlab_CON:RJHSE-5384(RJ45) -> Mlab_Pin_Headers:Straight_1x01
- moved J3 182.3 mm to (142.8, 127.7)
- moved M2 177.5 mm to (163.1, 128.1)
- moved M4 177.5 mm to (122.4, 128.1)
- moved J8 173.6 mm to (138.1, 87.5), turned to 180 degrees
- moved J7 170.1 mm to (145.7, 87.8), turned to 20 degrees
- moved M1 170.0 mm to (163.1, 87.5)
- moved M3 170.0 mm to (122.4, 87.5)
- moved J2 169.9 mm to (130.8, 88.1), turned to 0 degrees
- moved J1 147.7 mm to (130.9, 106.0), turned to -90 degrees
- renumbered J9 to J8
Connections:
- J2 pad 1: Net-(J1-Pad2) -> GND
- J3 pad 1: (no net) -> unconnected-(J3-Pad1)
- J3 pad 2: (no net) -> unconnected-(J3-Pad2)
- J3 pad 3: (no net) -> unconnected-(J3-Pad3)
- J3 pad 6: (no net) -> unconnected-(J3-Pad6)
- J3 pad 7: (no net) -> unconnected-(J3-Pad7)
- J3 pad 8: (no net) -> unconnected-(J3-Pad8)
- M1 pad 1: (no net) -> unconnected-(M1-Pad1)
- M2 pad 1: (no net) -> unconnected-(M2-Pad1)
- M3 pad 1: (no net) -> unconnected-(M3-Pad1)
- M4 pad 1: (no net) -> unconnected-(M4-Pad1)
Routing:
- net GND: track 153.7 -> 2.54 mm, vias 41 -> 6
- net /OUT1: track 69.1 -> 57.6 mm
- net Net-(J1-Pad8): track 34.8 -> 24.1 mm, vias 1 -> 0
- net Net-(J1-Pad2): track 34.5 -> 24.1 mm
- net Net-(J1-Pad7): track 33.9 -> 24.1 mm, vias 1 -> 0
- net Net-(J1-Pad3): track 33.8 -> 24.1 mm, vias 1 -> 0
- net Net-(J1-Pad6): track 33.2 -> 24.1 mm, vias 1 -> 0
- net Net-(J1-Pad4): track 33.0 -> 24.1 mm, vias 1 -> 0
- net Net-(J1-Pad5): track 32.2 -> 24.1 mm, vias 1 -> 0
- net /OUT2: track 72.6 -> 79.2 mm
Other:
- board size 50.3 x 40.1 mm -> 50.3 x 50.3 mm
- net class Default removed
- board text added: "2022"
- board text removed: "2017"
- board text removed: "OUT1"
